Commit message: Update materials and colors in URDF and fix package path in launch file

File: baxter_description/urdf/robots/baxter.urdf.xacro (robot description, xacro)
@@ -16,6 +16,6 @@
           <mesh filename="package://baxter_description/meshes/base/PEDESTAL.STL" scale="1 1 1" />
         </geometry>
-        <material name="lightgreen">
-          <color rgba=".047 .5843 .051 1" />
+        <material name="darkgray">
+          <color rgba=".2 .2 .2 1" />
         </material>
       </visual>
@@ -43,6 +43,6 @@
           <mesh filename="package://baxter_description/meshes/head/H0.STL" />
         </geometry>
-        <material name="yellow">
-          <color rgba="1 1 0 1" />
+        <material name="darkgray">
+          <color rgba=".2 .2 .2 1" />
         </material>
       </visual>
@@ -66,6 +66,6 @@
           <mesh filename="package://baxter_description/meshes/head/H1.STL" />
         </geometry>
-        <material name="yellow">
-          <color rgba="1 1 0 1" />
+        <material name="darkred">
+          <color rgba=".5 .1 .1 1" />
         </material>
       </visual>
@@ -112,6 +112,6 @@
           <mesh filename="package://baxter_description/meshes/torso/base_link.STL" />
         </geometry>
-        <material name="blue">
-          <color rgba="0 0 1 1" />
+        <material name="darkgray">
+          <color rgba=".2 .2 .2 1" />
         </material>
       </visual>
@@ -137,6 +137,6 @@
           <mesh filename="package://baxter_description/meshes/upper_shoulder/S0.STL" />
         </geometry>
-        <material name="blue">
-          <color rgba="0 0 1 1" />
+        <material name="darkgray">
+          <color rgba=".2 .2 .2 1" />
         </material>
       </visual>
@@ -164,6 +164,6 @@
           <mesh filename="package://baxter_description/meshes/lower_shoulder/S1.STL" />
         </geometry>
-        <material name="yellow">
-          <color rgba="1 1 0 1" />
+        <material name="darkred">
+          <color rgba=".5 .1 .1 1" />
         </material>
       </visual>
@@ -191,6 +191,6 @@
           <mesh filename="package://baxter_description/meshes/upper_elbow/E0.STL" />
         </geometry>
-        <material name="yellow">
-          <color rgba="1 1 0 1" />
+        <material name="darkred">
+          <color rgba=".5 .1 .1 1" />
         </material>
       </visual>
@@ -218,6 +218,6 @@
           <mesh filename="package://baxter_description/meshes/lower_elbow/E1.STL" />
         </geometry>
-        <material name="yellow">
-          <color rgba="1 1 0 1" />
+        <material name="darkred">
+          <color rgba=".5 .1 .1 1" />
         </material>
       </visual>
@@ -245,6 +245,6 @@
           <mesh filename="package://baxter_description/meshes/upper_forearm/W0.STL" />
         </geometry>
-        <material name="yellow">
-          <color rgba="1 1 0 1" />
+        <material name="darkred">
+          <color rgba=".5 .1 .1 1" />
         </material>
       </visual>
@@ -272,6 +272,6 @@
           <mesh filename="package://baxter_description/meshes/lower_forearm/W1.STL" />
         </geometry>
-        <material name="yellow">
-          <color rgba="1 1 0 1" />
+        <material name="darkgray">
+          <color rgba=".2 .2 .2 1" />
         </material>
       </visual>
@@ -299,6 +299,6 @@
           <mesh filename="package://baxter_description/meshes/wrist/W2.STL" />
         </geometry>
-        <material name="yellow">
-          <color rgba="1 1 0 1" />
+        <material name="darkred">
+          <color rgba=".5 .1 .1 1" />
         </material>
       </visual>
@@ -326,6 +326,6 @@
           <mesh filename="package://baxter_description/meshes/grippers/GRIPPER.STL" />
         </geometry>
-        <material name="yellow">
-          <color rgba="1 1 0 1" />
+        <material name="darkred">
+          <color rgba=".5 .1 .1 1" />
         </material>
       </visual>
@@ -350,6 +350,6 @@
           <mesh filename="package://baxter_description/meshes/upper_shoulder/S0.STL" />
         </geometry>
-        <material name="blue">
-          <color rgba="0 0 1 1" />
+        <material name="darkgray">
+          <color rgba=".2 .2 .2 1" />
         </material>
       </visual>
@@ -377,6 +377,6 @@
           <mesh filename="package://baxter_description/meshes/lower_shoulder/S1.STL" />
         </geometry>
-        <material name="yellow">
-          <color rgba="1 1 0 1" />
+        <material name="darkred">
+          <color rgba=".5 .1 .1 1" />
         </material>
       </visual>
@@ -404,6 +404,6 @@
           <mesh filename="package://baxter_description/meshes/upper_elbow/E0.STL" />
         </geometry>
-        <material name="yellow">
-          <color rgba="1 1 0 1" />
+        <material name="darkred">
+          <color rgba=".5 .1 .1 1" />
         </material>
       </visual>
@@ -431,6 +431,6 @@
           <mesh filename="package://baxter_description/meshes/lower_elbow/E1.STL" />
         </geometry>
-        <material name="yellow">
-          <color rgba="1 1 0 1" />
+        <material name="darkred">
+          <color rgba=".5 .1 .1 1" />
         </material>
       </visual>
@@ -458,6 +458,6 @@
           <mesh filename="package://baxter_description/meshes/upper_forearm/W0.STL" />
         </geometry>
-        <material name="yellow">
-          <color rgba="1 1 0 1" />
+        <material name="darkred">
+          <color rgba=".5 .1 .1 1" />
         </material>
       </visual>
@@ -485,6 +485,6 @@
           <mesh filename="package://baxter_description/meshes/lower_forearm/W1.STL" />
         </geometry>
-        <material name="yellow">
-          <color rgba="1 1 0 1" />
+        <material name="darkgray">
+          <color rgba=".2 .2 .2 1" />
         </material>
       </visual>
@@ -512,6 +512,6 @@
           <mesh filename="package://baxter_description/meshes/wrist/W2.STL" />
         </geometry>
-        <material name="yellow">
-          <color rgba="1 1 0 1" />
+        <material name="darkred">
+          <color rgba=".5 .1 .1 1" />
         </material>
       </visual>
@@ -539,6 +539,6 @@
           <mesh filename="package://baxter_description/meshes/grippers/GRIPPER.STL" />
         </geometry>
-        <material name="yellow">
-          <color rgba="1 1 0 1" />
+        <material name="darkred">
+          <color rgba=".5 .1 .1 1" />
         </material>
       </visual>
@@ -560,5 +560,5 @@
       <parent link="world" />
       <child link="base_link" />
-      <origin xyz="0 0 0" rpy="0 0 0" />
+      <origin xyz="0 0 .924" rpy="0 0 0" />
     </joint>
     <!-- head - screen -->
@@ -726,4 +726,5 @@
     </xacro:if>
   </xacro:macro>
-  <!--xacro:baxter name="baxter" /-->
+  <!--xacro:baxter
+  name="baxter" /-->
 </robot>

Commit message: Refactor sensor configurations in URDF files and update Gazebo launch parameters

File: baxter_description/urdf/robots/baxter.urdf.xacro (robot description, xacro)
@@ -722,6 +722,6 @@
     <xacro:if value="${use_sensors}">
       <xacro:imu parent="base_link" frame="imu_link" />
-      <xacro:lidar parent="base_link" frame="lidar_link" />
-      <xacro:camera_color parent="base_link" frame="camera_link" />
+      <xacro:lidar parent="hat" frame="lidar_link" />
+      <xacro:camera_color parent="screen" frame="camera_link" />
     </xacro:if>
   </xacro:macro>

File: baxter_description/urdf/sensors/camera_color.urdf.xacro (robot description, xacro)
@@ -4,17 +4,20 @@
     <link name="${frame}">
       <visual>
+        <origin rpy="0 1.5708 0" xyz="0 0 0" />
         <geometry>
-          <box size="0.05 0.05 0.05" />
+          <cylinder length="0.005" radius="0.009" />
         </geometry>
+        <material name="cam_lens">
+          <color rgba="0.05 0.05 0.05 1" />
+        </material>
       </visual>
       <collision>
+        <origin rpy="0 1.5708 0" xyz="0 0 0" />
         <geometry>
-          <box size="0.05 0.05 0.05" />
+          <box size="0.04 0.025 0.02" />
         </geometry>
       </collision>
       <inertial>
-        <!-- TODO_FILL_MASS -->
         <mass value="0.1" />
-        <!-- TODO_FILL_INERTIA -->
         <inertia ixx="1e-3" ixy="0.0" ixz="0.0" iyy="1e-3" iyz="0.0" izz="1e-3"/>
       </inertial>
@@ -23,5 +26,5 @@
       <parent link="${parent}" />
       <child link="${frame}" />
-      <origin rpy="0 0 0" xyz=".15 0 .3" />
+      <origin rpy="0 .26 0" xyz=".05 0 .065" />
     </joint>
   </xacro:macro>

File: baxter_description/urdf/sensors/lidar.urdf.xacro (robot description, xacro)
@@ -4,24 +4,27 @@
     <link name="${frame}">
       <visual>
+        <origin rpy="0 0 0" xyz="0 0 0" />
         <geometry>
-          <cylinder length="0.05" radius="0.04" />
+          <cylinder length="0.01" radius="0.01" />
         </geometry>
+        <material name="lidar_black">
+          <color rgba="0.1 0.1 0.1 1" />
+        </material>
       </visual>
       <collision>
+        <origin rpy="0 0 0" xyz="0 0 0" />
         <geometry>
-          <cylinder length="0.05" radius="0.04" />
+          <cylinder length="0.01" radius="0.01" />
         </geometry>
       </collision>
       <inertial>
-        <!-- TODO_FILL_MASS -->
         <mass value=".2" />
-        <!-- TODO_FILL_INERTIA -->
         <inertia ixx="1e-4" ixy="0.0" ixz="0.0" iyy="1e-4" iyz="0.0" izz="1e-4"/>
-        </inertial>
+      </inertial>
     </link>
     <joint name="${frame}_joint" type="fixed">
       <parent link="${parent}" />
       <child link="${frame}" />
-      <origin rpy="0 0 0" xyz="0 0 .5" />
+      <origin rpy="0 0 0" xyz="0 0 .04" />
     </joint>
   </xacro:macro>

File: gazebo_baxter/urdf/sensors/lidar_gazebo.urdf.xacro (robot description, xacro)
@@ -3,5 +3,5 @@
     <xacro:macro name="lidar_gazebo" params="frame topic_name:=scan sensor_name:=lidar_sensor">
         <gazebo reference="${frame}">
-            <sensor name="${sensor_name}" type="gpu_ray">
+            <sensor name="${sensor_name}" type="gpu_lidar">
                 <pose>0 0 0 0 0 0</pose>
                 <always_on>true</always_on>
@@ -9,5 +9,5 @@
                 <visualize>true</visualize>
                 <topic>${topic_name}</topic>
-                <ray>
+                <lidar>
                     <scan>
                         <horizontal>
@@ -28,5 +28,5 @@
                         <stddev>0.01</stddev>
                     </noise>
-                </ray>
+                </lidar>
             </sensor>
         </gazebo>
