Commit message: Add electric gripper components and update robot URDF
- Introduced new XACRO files for electric gripper finger tips: basic_hard_tip.xacro, extended_narrow.xacro, and paddle_tip.xacro.
- Updated baxter.urdf.xacro to include the electric gripper and its components.
- Refactored existing links and joints for clarity and consistency.

File: baxter_description/urdf/robots/baxter.urdf.xacro (robot description, xacro)
@@ -6,4 +6,7 @@
   <xacro:include filename="$(find baxter_description)/urdf/sensors/camera_color.urdf.xacro" />
   <xacro:include filename="$(find baxter_description)/urdf/sensors/camera_rgbd.urdf.xacro" />
+  <!-- Include electric gripper -->
+  <xacro:include
+    filename="$(find baxter_description)/urdf/electric_gripper/baxter_electric_gripper.xacro" />
   <!-- Macro definition -->
   <xacro:macro name="baxter" params="name use_sensors:=true">
@@ -23,6 +26,5 @@
         <origin rpy="0 0 0" xyz="0 0 0" />
         <geometry>
-          <mesh
-            filename="package://baxter_description/meshes/base/pedestal_link_collision.STL"
+          <mesh filename="package://baxter_description/meshes/base/pedestal_link_collision.STL"
             scale="1 1 1" />
         </geometry>
@@ -32,6 +34,5 @@
         <mass value="60.86397744" />
         <inertia ixx="5.0635929" ixy="0.00103417" ixz="0.80199628" iyy="6.08689388"
-          iyz="0.00105311"
-          izz="4.96191932" />
+          iyz="0.00105311" izz="4.96191932" />
       </inertial>
     </link>
@@ -125,10 +126,8 @@
         <mass value="35.336455" />
         <inertia ixx="1.849155" ixy="-0.000354" ixz="-0.154188" iyy="1.662671"
-          iyz="0.003292"
-          izz="0.802239" />
+          iyz="0.003292" izz="0.802239" />
       </inertial>
     </link>
     <!-- ====== LEFT ARM LINKS ====== -->
-    <!-- Left upper shoulder -->
     <link name="left_upper_shoulder">
       <visual>
@@ -144,6 +143,4 @@
         <origin rpy="0 0 1.5708" xyz="0 0 0" />
         <geometry>
-          <!--cylinder
-          length="0.2722" radius="0.06" /-->
           <mesh filename="package://baxter_description/meshes/upper_shoulder/S0.STL" />
         </geometry>
@@ -153,9 +150,7 @@
         <mass value="5.70044" />
         <inertia ixx="0.04709102262" ixy="0.00012787556" ixz="0.00614870039"
-          iyy="0.03766976455"
-          iyz="0.00078086899" izz="0.03595988478" />
-      </inertial>
-    </link>
-    <!-- Left lower shoulder -->
+          iyy="0.03766976455" iyz="0.00078086899" izz="0.03595988478" />
+      </inertial>
+    </link>
     <link name="left_lower_shoulder">
       <visual>
@@ -171,6 +166,4 @@
         <origin rpy="1.5708 0 1.5708" xyz="0 0 0" />
         <geometry>
-          <!--cylinder
-          length="0.12" radius="0.06" /-->
           <mesh filename="package://baxter_description/meshes/lower_shoulder/S1.STL" />
         </geometry>
@@ -180,9 +173,7 @@
         <mass value="3.22698" />
         <inertia ixx="0.01175209419" ixy="-0.00030096398" ixz="0.00207675762"
-          iyy="0.0278859752"
-          iyz="-0.00018821993" izz="0.02078749298" />
-      </inertial>
-    </link>
-    <!-- Left upper elbow -->
+          iyy="0.0278859752" iyz="-0.00018821993" izz="0.02078749298" />
+      </inertial>
+    </link>
     <link name="left_upper_elbow">
       <visual>
@@ -198,6 +189,4 @@
         <origin rpy="1.5708 1.5708 3.1416" xyz="0 0 0" />
         <geometry>
-          <!--cylinder
-          length="0.107" radius="0.06" /-->
           <mesh filename="package://baxter_description/meshes/upper_elbow/E0.STL" />
         </geometry>
@@ -207,9 +196,7 @@
         <mass value="4.31272" />
         <inertia ixx="0.02661733557" ixy="0.00029270634" ixz="0.00392189887"
-          iyy="0.02844355207"
-          iyz="0.0010838933" izz="0.01248008322" />
-      </inertial>
-    </link>
-    <!-- Left lower elbow -->
+          iyy="0.02844355207" iyz="0.0010838933" izz="0.01248008322" />
+      </inertial>
+    </link>
     <link name="left_lower_elbow">
       <visual>
@@ -225,6 +212,4 @@
         <origin rpy="-1.5708 1.5708 1.5708" xyz="0 0 0" />
         <geometry>
-          <!--cylinder
-          length="0.10" radius="0.06" /-->
           <mesh filename="package://baxter_description/meshes/lower_elbow/E1.STL" />
         </geometry>
@@ -234,9 +219,7 @@
         <mass value="2.07206" />
         <inertia ixx="0.00711582686" ixy="0.00036036173" ixz="0.0007459496"
-          iyy="0.01318227876"
-          iyz="-0.00019663418" izz="0.00926852064" />
-      </inertial>
-    </link>
-    <!-- Left upper forearm -->
+          iyy="0.01318227876" iyz="-0.00019663418" izz="0.00926852064" />
+      </inertial>
+    </link>
     <link name="left_upper_forearm">
       <visual>
@@ -252,6 +235,4 @@
         <origin rpy="3.1416 0 -1.5708" xyz="0 0 0" />
         <geometry>
-          <!--cylinder
-          length="0.088" radius="0.06" /-->
           <mesh filename="package://baxter_description/meshes/upper_forearm/W0.STL" />
         </geometry>
@@ -261,9 +242,7 @@
         <mass value="2.24665" />
         <inertia ixx="0.01667742825" ixy="0.00018403705" ixz="0.00018657629"
-          iyy="0.01675457264"
-          iyz="-0.00064732352" izz="0.0037463115" />
-      </inertial>
-    </link>
-    <!-- Left lower forearm -->
+          iyy="0.01675457264" iyz="-0.00064732352" izz="0.0037463115" />
+      </inertial>
+    </link>
     <link name="left_lower_forearm">
       <visual>
@@ -279,6 +258,4 @@
         <origin rpy="0 1.5708 0" xyz="0 0 0" />
         <geometry>
-          <!--cylinder
-          length="0.10" radius="0.06" /-->
           <mesh filename="package://baxter_description/meshes/lower_forearm/W1.STL" />
         </geometry>
@@ -288,12 +265,10 @@
         <mass value="1.60979" />
         <inertia ixx="0.00387607152" ixy="-0.00044384784" ixz="-0.00021115038"
-          iyy="0.00700537914"
-          iyz="0.00015348067" izz="0.0055275524" />
-      </inertial>
-    </link>
-    <!-- Left wrist -->
+          iyy="0.00700537914" iyz="0.00015348067" izz="0.0055275524" />
+      </inertial>
+    </link>
     <link name="left_wrist">
       <visual>
-        <origin rpy="0 3.1416 -1.5708" xyz="0 0 0" />
+        <origin rpy="0 3.1416 0" xyz="0 0 0" />
         <geometry>
           <mesh filename="package://baxter_description/meshes/wrist/W2.STL" />
@@ -304,44 +279,17 @@
       </visual>
       <collision>
-        <origin rpy="0 3.1416 -1.5708" xyz="0 0 0" />
-        <geometry>
-          <!--cylinder
-          length="0.165" radius="0.06" /-->
+        <origin rpy="0 3.1416 0" xyz="0 0 0" />
+        <geometry>
           <mesh filename="package://baxter_description/meshes/wrist/W2.STL" />
         </geometry>
       </collision>
       <inertial>
-        <origin rpy="0 3.1416 -1.5708" xyz="0 0 0" />
+        <origin rpy="0 3.1416 0" xyz="0 0 0" />
         <mass value="0.35093" />
         <inertia ixx="0.00025289155" ixy="0.00000575311" ixz="-0.00000159345"
-          iyy="0.0002688601"
-          iyz="-0.00000519818" izz="0.0003074118" />
-      </inertial>
-    </link>
-    <!-- Left grippers -->
-    <link name="left_grippers">
-      <visual>
-        <origin rpy="0 3.1416 0" xyz="0 0 0" />
-        <geometry>
-          <mesh filename="package://baxter_description/meshes/grippers/GRIPPER.STL" />
-        </geometry>
-        <material name="darkred">
-          <color rgba=".5 .1 .1 1" />
-        </material>
-      </visual>
-      <collision>
-        <origin rpy="0 3.1416 0" xyz="0 0 0" />
-        <geometry>
-          <mesh filename="package://baxter_description/meshes/grippers/GRIPPER.STL" />
-        </geometry>
-      </collision>
-      <inertial>
-        <origin rpy="0 3.1416 0" xyz="0 0 0" />
-        <mass value=".5" />
-        <inertia ixx="0.01" ixy="0.0" ixz="0.0" iyy="0.01" iyz="0.0" izz="0.01" />
+          iyy="0.0002688601" iyz="-0.00000519818" izz="0.0003074118" />
       </inertial>
     </link>
     <!-- ====== RIGHT ARM LINKS ====== -->
-    <!-- Right upper shoulder -->
     <link name="right_upper_shoulder">
       <visual>
@@ -357,6 +305,4 @@
         <origin rpy="0 0 -1.5708" xyz="0 0 0" />
         <geometry>
-          <!--cylinder
-          length="0.2722" radius="0.06" /-->
           <mesh filename="package://baxter_description/meshes/upper_shoulder/S0.STL" />
         </geometry>
@@ -366,9 +312,7 @@
         <mass value="5.70044" />
         <inertia ixx="0.04709102262" ixy="0.00012787556" ixz="0.00614870039"
-          iyy="0.03766976455"
-          iyz="0.00078086899" izz="0.03595988478" />
-      </inertial>
-    </link>
-    <!-- Right lower shoulder -->
+          iyy="0.03766976455" iyz="0.00078086899" izz="0.03595988478" />
+      </inertial>
+    </link>
     <link name="right_lower_shoulder">
       <visual>
@@ -384,6 +328,4 @@
         <origin rpy="1.5708 0 -1.5708" xyz="0 0 0" />
         <geometry>
-          <!--cylinder
-          length="0.12" radius="0.06" /-->
           <mesh filename="package://baxter_description/meshes/lower_shoulder/S1.STL" />
         </geometry>
@@ -393,9 +335,7 @@
         <mass value="3.22698" />
         <inertia ixx="0.01175209419" ixy="-0.00030096398" ixz="0.00207675762"
-          iyy="0.0278859752"
-          iyz="-0.00018821993" izz="0.02078749298" />
-      </inertial>
-    </link>
-    <!-- Right upper elbow -->
+          iyy="0.0278859752" iyz="-0.00018821993" izz="0.02078749298" />
+      </inertial>
+    </link>
     <link name="right_upper_elbow">
       <visual>
@@ -411,6 +351,4 @@
         <origin rpy="0 1.5708 -1.5708" xyz="0 0 0" />
         <geometry>
-          <!--cylinder
-          length="0.107" radius="0.06" /-->
           <mesh filename="package://baxter_description/meshes/upper_elbow/E0.STL" />
         </geometry>
@@ -420,9 +358,7 @@
         <mass value="4.31272" />
         <inertia ixx="0.02661733557" ixy="0.00029270634" ixz="0.00392189887"
-          iyy="0.02844355207"
-          iyz="0.0010838933" izz="0.01248008322" />
-      </inertial>
-    </link>
-    <!-- Right lower elbow -->
+          iyy="0.02844355207" iyz="0.0010838933" izz="0.01248008322" />
+      </inertial>
+    </link>
     <link name="right_lower_elbow">
       <visual>
@@ -438,6 +374,4 @@
         <origin rpy="-1.5708 1.5708 1.5708" xyz="0 0 0" />
         <geometry>
-          <!--cylinder
-          length="0.10" radius="0.06" /-->
           <mesh filename="package://baxter_description/meshes/lower_elbow/E1.STL" />
         </geometry>
@@ -447,9 +381,7 @@
         <mass value="2.07206" />
         <inertia ixx="0.00711582686" ixy="0.00036036173" ixz="0.0007459496"
-          iyy="0.01318227876"
-          iyz="-0.00019663418" izz="0.00926852064" />
-      </inertial>
-    </link>
-    <!-- Right upper forearm -->
+          iyy="0.01318227876" iyz="-0.00019663418" izz="0.00926852064" />
+      </inertial>
+    </link>
     <link name="right_upper_forearm">
       <visual>
@@ -465,6 +397,4 @@
         <origin rpy="3.1416 0 1.5708" xyz="0 0 0" />
         <geometry>
-          <!--cylinder
-          length="0.088" radius="0.06" /-->
           <mesh filename="package://baxter_description/meshes/upper_forearm/W0.STL" />
         </geometry>
@@ -474,9 +404,7 @@
         <mass value="2.24665" />
         <inertia ixx="0.01667742825" ixy="0.00018403705" ixz="0.00018657629"
-          iyy="0.01675457264"
-          iyz="-0.00064732352" izz="0.0037463115" />
-      </inertial>
-    </link>
-    <!-- Right_lower forearm -->
+          iyy="0.01675457264" iyz="-0.00064732352" izz="0.0037463115" />
+      </inertial>
+    </link>
     <link name="right_lower_forearm">
       <visual>
@@ -492,6 +420,4 @@
         <origin rpy="0 1.5708 -3.1416" xyz="0 0 0" />
         <geometry>
-          <!--cylinder
-          length="0.10" radius="0.06" /-->
           <mesh filename="package://baxter_description/meshes/lower_forearm/W1.STL" />
         </geometry>
@@ -501,59 +427,30 @@
         <mass value="1.60979" />
         <inertia ixx="0.00387607152" ixy="-0.00044384784" ixz="-0.00021115038"
-          iyy="0.00700537914"
-          iyz="0.00015348067" izz="0.0055275524" />
-      </inertial>
-    </link>
-    <!-- Right wrist -->
+          iyy="0.00700537914" iyz="0.00015348067" izz="0.0055275524" />
+      </inertial>
+    </link>
     <link name="right_wrist">
       <visual>
+        <origin rpy="0 3.1416 0" xyz="0 0 0" />
+        <geometry>
+          <mesh filename="package://baxter_description/meshes/wrist/W2.STL" />
+        </geometry>
+        <material name="darkred">
+          <color rgba=".5 .1 .1 1" />
+        </material>
+      </visual>
+      <collision>
         <origin rpy="0 3.1416 1.5708" xyz="0 0 0" />
         <geometry>
           <mesh filename="package://baxter_description/meshes/wrist/W2.STL" />
         </geometry>
-        <material name="darkred">
-          <color rgba=".5 .1 .1 1" />
-        </material>
-      </visual>
-      <collision>
-        <origin rpy="0 3.1416 1.5708" xyz="0 0 0" />
-        <geometry>
-          <!--cylinder
-          length="0.165" radius="0.06" /-->
-          <mesh filename="package://baxter_description/meshes/wrist/W2.STL" />
-        </geometry>
-      </collision>
-      <inertial>
-        <origin rpy="0 3.1416 1.5708" xyz="0 0 0" />
+      </collision>
+      <inertial>
+        <origin rpy="0 3.1416 1.5708" xyz="0.00198 0.00125 0.01855"/>
         <mass value="0.35093" />
         <inertia ixx="0.00025289155" ixy="0.00000575311" ixz="-0.00000159345"
-          iyy="0.0002688601"
-          iyz="-0.00000519818" izz="0.0003074118" />
-      </inertial>
-    </link>
-    <!-- Right grippers -->
-    <link name="right_grippers">
-      <visual>
-        <origin rpy="0 -3.1416 0" xyz="0 0 0" />
-        <geometry>
-          <mesh filename="package://baxter_description/meshes/grippers/GRIPPER.STL" />
-        </geometry>
-        <material name="darkred">
-          <color rgba=".5 .1 .1 1" />
-        </material>
-      </visual>
-      <collision>
-        <origin rpy="0 -3.1416 0" xyz="0 0 0" />
-        <geometry>
-          <mesh filename="package://baxter_description/meshes/grippers/GRIPPER.STL" />
-        </geometry>
-      </collision>
-      <inertial>
-        <origin rpy="0 -3.1416 0" xyz="0 0 0" />
-        <mass value=".5" />
-        <inertia ixx="0.01" ixy="0.0" ixz="0.0" iyy="0.01" iyz="0.0" izz="0.01" />
-      </inertial>
-    </link>
-    <!-- TODO: Add joints/links for baxter (arms, wheels, etc.) -->
+          iyy="0.0002688601" iyz="-0.00000519818" izz="0.0003074118" />
+      </inertial>
+    </link>
     <!-- ====== JOINTS ====== -->
     <joint name="world_to_base" type="fixed">
@@ -562,5 +459,4 @@
       <origin xyz="0 0 .924" rpy="0 0 0" />
     </joint>
-    <!-- head - screen -->
     <joint name="head_screen" type="fixed">
       <origin rpy="0 0 0" xyz=".07 0 0" />
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