Commit message: Add extended narrow STL model and update URDF references for electric gripper

File: baxter_description/urdf/electric_gripper/baxter_electric_gripper.xacro (robot description, xacro)
@@ -1,26 +1,18 @@
 <?xml version="1.0"?>
 <robot xmlns:xacro="http://www.ros.org/wiki/xacro" name="baxter_electric_gripper">
-    <!--
-    Gripper eléctrico de Baxter — autocontenido en baxter_description.
-    Equivalente funcional de rethink_electric_gripper.xacro pero sin
-    depender del paquete rethink_ee_description.
-    Parámetros:
-      side           — "left" o "right"
-      l_finger       — tipo de dedo izquierdo  (e.g. "extended_narrow")
-      l_finger_slot  — slot 1 o 2
-      l_finger_tip   — tipo de tip izquierdo   (e.g. "paddle_tip")
-      l_finger_grasp — "inner" o "outer"
-      r_finger / r_finger_slot / r_finger_tip / r_finger_grasp — igual para el derecho
-    Requiere que el link "${side}_hand" ya exista en el URDF padre.
-  -->
     <xacro:macro name="baxter_electric_gripper"
         params="side
-                       l_finger l_finger_slot l_finger_tip l_finger_grasp
-                       r_finger r_finger_slot r_finger_tip r_finger_grasp">
+        l_finger l_finger_slot l_finger_tip l_finger_grasp
+        r_finger r_finger_slot r_finger_tip r_finger_grasp">
         <xacro:property name="gripper_side" value="${side[0]}" scope="local" />
         <!-- ===== BASE DEL GRIPPER ===== -->
         <link name="${side}_gripper_base">
             <visual>
-                <origin rpy="${-pi/2} ${pi} 0" xyz="0 0 0" />
+                <!-- <origin rpy="${-pi/2} ${pi} 0" xyz="0 0 0" /> -->
+                <origin rpy="${pi/2} 0 ${pi}" xyz="0 0 0" />
+                <geometry>
+                    <mesh
+                        filename="package://baxter_description/meshes/electric_gripper/electric_gripper_base.DAE" />
+                </geometry>
                 <geometry>
                     <mesh

File: baxter_description/urdf/electric_gripper/fingers/extended_narrow.xacro (robot description, xacro)
@@ -10,5 +10,5 @@
                 <geometry>
                     <mesh
-                        filename="package://baxter_description/meshes/electric_gripper/fingers/extended_narrow.DAE" />
+                        filename="package://baxter_description/meshes/electric_gripper/fingers/extended_narrow.STL" />
                 </geometry>
             </visual>
@@ -24,5 +24,5 @@
                 </geometry>
             </collision>
-            <!-- Nudillo -->
+            <!-- knuckle -->
             <xacro:property name="knuckle_box_height" value="0.01" scope="local" />
             <xacro:property name="knuckle_box_width" value="0.017" scope="local" />

File: baxter_description/urdf/robots/baxter.urdf.xacro (robot description, xacro)
@@ -129,4 +129,174 @@
       </inertial>
     </link>
+    <!-- ====== RIGHT ARM LINKS ====== -->
+    <link name="right_upper_shoulder">
+      <visual>
+        <origin rpy="0 0 -1.5708" xyz="0 0 0" />
+        <geometry>
+          <mesh filename="package://baxter_description/meshes/upper_shoulder/S0.STL" />
+        </geometry>
+        <material name="darkgray">
+          <color rgba=".2 .2 .2 1" />
+        </material>
+      </visual>
+      <collision>
+        <origin rpy="0 0 -1.5708" xyz="0 0 0" />
+        <geometry>
+          <mesh filename="package://baxter_description/meshes/upper_shoulder/S0.STL" />
+        </geometry>
+      </collision>
+      <inertial>
+        <origin rpy="0 0 -1.5708" xyz="0 0 0" />
+        <mass value="5.70044" />
+        <inertia ixx="0.04709102262" ixy="0.00012787556" ixz="0.00614870039"
+          iyy="0.03766976455" iyz="0.00078086899" izz="0.03595988478" />
+      </inertial>
+    </link>
+    <link name="right_lower_shoulder">
+      <visual>
+        <origin rpy="1.5708 0 -1.5708" xyz="0 0 0" />
+        <geometry>
+          <mesh filename="package://baxter_description/meshes/lower_shoulder/S1.STL" />
+        </geometry>
+        <material name="darkred">
+          <color rgba=".5 .1 .1 1" />
+        </material>
+      </visual>
+      <collision>
+        <origin rpy="1.5708 0 -1.5708" xyz="0 0 0" />
+        <geometry>
+          <mesh filename="package://baxter_description/meshes/lower_shoulder/S1.STL" />
+        </geometry>
+      </collision>
+      <inertial>
+        <origin rpy="1.5708 0 -1.5708" xyz="0 0 0" />
+        <mass value="3.22698" />
+        <inertia ixx="0.01175209419" ixy="-0.00030096398" ixz="0.00207675762"
+          iyy="0.0278859752" iyz="-0.00018821993" izz="0.02078749298" />
+      </inertial>
+    </link>
+    <link name="right_upper_elbow">
+      <visual>
+        <origin rpy="0 1.5708 -1.5708" xyz="0 0 0" />
+        <geometry>
+          <mesh filename="package://baxter_description/meshes/upper_elbow/E0.STL" />
+        </geometry>
+        <material name="darkred">
+          <color rgba=".5 .1 .1 1" />
+        </material>
+      </visual>
+      <collision>
+        <origin rpy="0 1.5708 -1.5708" xyz="0 0 0" />
+        <geometry>
+          <mesh filename="package://baxter_description/meshes/upper_elbow/E0.STL" />
+        </geometry>
+      </collision>
+      <inertial>
+        <origin rpy="0 1.5708 -1.5708" xyz="0 0 0" />
+        <mass value="4.31272" />
+        <inertia ixx="0.02661733557" ixy="0.00029270634" ixz="0.00392189887"
+          iyy="0.02844355207" iyz="0.0010838933" izz="0.01248008322" />
+      </inertial>
+    </link>
+    <link name="right_lower_elbow">
+      <visual>
+        <origin rpy="-1.5708 1.5708 1.5708" xyz="0 0 0" />
+        <geometry>
+          <mesh filename="package://baxter_description/meshes/lower_elbow/E1.STL" />
+        </geometry>
+        <material name="darkred">
+          <color rgba=".5 .1 .1 1" />
+        </material>
+      </visual>
+      <collision>
+        <origin rpy="-1.5708 1.5708 1.5708" xyz="0 0 0" />
+        <geometry>
+          <mesh filename="package://baxter_description/meshes/lower_elbow/E1.STL" />
+        </geometry>
+      </collision>
+      <inertial>
+        <origin rpy="-1.5708 1.5708 1.5708" xyz="0 0 0" />
+        <mass value="2.07206" />
+        <inertia ixx="0.00711582686" ixy="0.00036036173" ixz="0.0007459496"
+          iyy="0.01318227876" iyz="-0.00019663418" izz="0.00926852064" />
+      </inertial>
+    </link>
+    <link name="right_upper_forearm">
+      <visual>
+        <origin rpy="3.1416 0 1.5708" xyz="0 0 0" />
+        <geometry>
+          <mesh filename="package://baxter_description/meshes/upper_forearm/W0.STL" />
+        </geometry>
+        <material name="darkred">
+          <color rgba=".5 .1 .1 1" />
+        </material>
+      </visual>
+      <collision>
+        <origin rpy="3.1416 0 1.5708" xyz="0 0 0" />
+        <geometry>
+          <mesh filename="package://baxter_description/meshes/upper_forearm/W0.STL" />
+        </geometry>
+      </collision>
+      <inertial>
+        <origin rpy="3.1416 0 1.5708" xyz="0 0 0" />
+        <mass value="2.24665" />
+        <inertia ixx="0.01667742825" ixy="0.00018403705" ixz="0.00018657629"
+          iyy="0.01675457264" iyz="-0.00064732352" izz="0.0037463115" />
+      </inertial>
+    </link>
+    <link name="right_lower_forearm">
+      <visual>
+        <origin rpy="0 1.5708 -3.1416" xyz="0 0 0" />
+        <geometry>
+          <mesh filename="package://baxter_description/meshes/lower_forearm/W1.STL" />
+        </geometry>
+        <material name="darkgray">
+          <color rgba=".2 .2 .2 1" />
+        </material>
+      </visual>
+      <collision>
+        <origin rpy="0 1.5708 -3.1416" xyz="0 0 0" />
+        <geometry>
+          <mesh filename="package://baxter_description/meshes/lower_forearm/W1.STL" />
+        </geometry>
+      </collision>
+      <inertial>
+        <origin rpy="0 1.5708 -3.1416" xyz="0 0 0" />
+        <mass value="1.60979" />
+        <inertia ixx="0.00387607152" ixy="-0.00044384784" ixz="-0.00021115038"
+          iyy="0.00700537914" iyz="0.00015348067" izz="0.0055275524" />
+      </inertial>
+    </link>
+    <link name="right_wrist">
+      <visual>
+        <origin rpy="0 3.1416 0" xyz="0 0 0" />
+        <geometry>
+          <mesh filename="package://baxter_description/meshes/wrist/W2.STL" />
+        </geometry>
+        <material name="darkred">
+          <color rgba=".5 .1 .1 1" />
+        </material>
+      </visual>
+      <collision>
+        <origin rpy="0 3.1416 1.5708" xyz="0 0 0" />
+        <geometry>
+          <mesh filename="package://baxter_description/meshes/wrist/W2.STL" />
+        </geometry>
+      </collision>
+      <inertial>
+        <origin rpy="0 3.1416 1.5708" xyz="0.00198 0.00125 0.01855" />
+        <mass value="0.35093" />
+        <inertia ixx="0.00025289155" ixy="0.00000575311" ixz="-0.00000159345"
+          iyy="0.0002688601" iyz="-0.00000519818" izz="0.0003074118" />
+      </inertial>
+    </link>
+    <!-- right_hand -->
+    <link name="right_hand">
+      <inertial>
+        <origin rpy="0 0 0" xyz="0 0 0" />
+        <mass value="0.0001" />
+        <inertia ixx="1e-08" ixy="0" ixz="0" iyy="1e-08" iyz="0" izz="1e-08" />
+      </inertial>
+    </link>
     <!-- ====== LEFT ARM LINKS ====== -->
     <link name="left_upper_shoulder">
@@ -291,164 +461,10 @@
       </inertial>
     </link>
-    <!-- ====== RIGHT ARM LINKS ====== -->
-    <link name="right_upper_shoulder">
-      <visual>
-        <origin rpy="0 0 -1.5708" xyz="0 0 0" />
-        <geometry>
-          <mesh filename="package://baxter_description/meshes/upper_shoulder/S0.STL" />
-        </geometry>
-        <material name="darkgray">
-          <color rgba=".2 .2 .2 1" />
-        </material>
-      </visual>
-      <collision>
-        <origin rpy="0 0 -1.5708" xyz="0 0 0" />
-        <geometry>
-          <mesh filename="package://baxter_description/meshes/upper_shoulder/S0.STL" />
-        </geometry>
-      </collision>
-      <inertial>
-        <origin rpy="0 0 -1.5708" xyz="0 0 0" />
-        <mass value="5.70044" />
-        <inertia ixx="0.04709102262" ixy="0.00012787556" ixz="0.00614870039"
-          iyy="0.03766976455" iyz="0.00078086899" izz="0.03595988478" />
-      </inertial>
-    </link>
-    <link name="right_lower_shoulder">
-      <visual>
-        <origin rpy="1.5708 0 -1.5708" xyz="0 0 0" />
-        <geometry>
-          <mesh filename="package://baxter_description/meshes/lower_shoulder/S1.STL" />
-        </geometry>
-        <material name="darkred">
-          <color rgba=".5 .1 .1 1" />
-        </material>
-      </visual>
-      <collision>
-        <origin rpy="1.5708 0 -1.5708" xyz="0 0 0" />
-        <geometry>
-          <mesh filename="package://baxter_description/meshes/lower_shoulder/S1.STL" />
-        </geometry>
-      </collision>
-      <inertial>
-        <origin rpy="1.5708 0 -1.5708" xyz="0 0 0" />
-        <mass value="3.22698" />
-        <inertia ixx="0.01175209419" ixy="-0.00030096398" ixz="0.00207675762"
-          iyy="0.0278859752" iyz="-0.00018821993" izz="0.02078749298" />
-      </inertial>
-    </link>
-    <link name="right_upper_elbow">
-      <visual>
-        <origin rpy="0 1.5708 -1.5708" xyz="0 0 0" />
-        <geometry>
-          <mesh filename="package://baxter_description/meshes/upper_elbow/E0.STL" />
-        </geometry>
-        <material name="darkred">
-          <color rgba=".5 .1 .1 1" />
-        </material>
-      </visual>
-      <collision>
-        <origin rpy="0 1.5708 -1.5708" xyz="0 0 0" />
-        <geometry>
-          <mesh filename="package://baxter_description/meshes/upper_elbow/E0.STL" />
-        </geometry>
-      </collision>
-      <inertial>
-        <origin rpy="0 1.5708 -1.5708" xyz="0 0 0" />
-        <mass value="4.31272" />
-        <inertia ixx="0.02661733557" ixy="0.00029270634" ixz="0.00392189887"
-          iyy="0.02844355207" iyz="0.0010838933" izz="0.01248008322" />
-      </inertial>
-    </link>
-    <link name="right_lower_elbow">
-      <visual>
-        <origin rpy="-1.5708 1.5708 1.5708" xyz="0 0 0" />
-        <geometry>
-          <mesh filename="package://baxter_description/meshes/lower_elbow/E1.STL" />
-        </geometry>
-        <material name="darkred">
-          <color rgba=".5 .1 .1 1" />
-        </material>
-      </visual>
-      <collision>
-        <origin rpy="-1.5708 1.5708 1.5708" xyz="0 0 0" />
-        <geometry>
-          <mesh filename="package://baxter_description/meshes/lower_elbow/E1.STL" />
-        </geometry>
-      </collision>
-      <inertial>
-        <origin rpy="-1.5708 1.5708 1.5708" xyz="0 0 0" />
-        <mass value="2.07206" />
-        <inertia ixx="0.00711582686" ixy="0.00036036173" ixz="0.0007459496"
-          iyy="0.01318227876" iyz="-0.00019663418" izz="0.00926852064" />
-      </inertial>
-    </link>
-    <link name="right_upper_forearm">
-      <visual>
-        <origin rpy="3.1416 0 1.5708" xyz="0 0 0" />
-        <geometry>
-          <mesh filename="package://baxter_description/meshes/upper_forearm/W0.STL" />
-        </geometry>
-        <material name="darkred">
-          <color rgba=".5 .1 .1 1" />
-        </material>
-      </visual>
-      <collision>
-        <origin rpy="3.1416 0 1.5708" xyz="0 0 0" />
-        <geometry>
-          <mesh filename="package://baxter_description/meshes/upper_forearm/W0.STL" />
-        </geometry>
-      </collision>
-      <inertial>
-        <origin rpy="3.1416 0 1.5708" xyz="0 0 0" />
-        <mass value="2.24665" />
-        <inertia ixx="0.01667742825" ixy="0.00018403705" ixz="0.00018657629"
-          iyy="0.01675457264" iyz="-0.00064732352" izz="0.0037463115" />
-      </inertial>
-    </link>
-    <link name="right_lower_forearm">
-      <visual>
-        <origin rpy="0 1.5708 -3.1416" xyz="0 0 0" />
-        <geometry>
-          <mesh filename="package://baxter_description/meshes/lower_forearm/W1.STL" />
-        </geometry>
-        <material name="darkgray">
-          <color rgba=".2 .2 .2 1" />
-        </material>
-      </visual>
-      <collision>
-        <origin rpy="0 1.5708 -3.1416" xyz="0 0 0" />
-        <geometry>
-          <mesh filename="package://baxter_description/meshes/lower_forearm/W1.STL" />
-        </geometry>
-      </collision>
-      <inertial>
-        <origin rpy="0 1.5708 -3.1416" xyz="0 0 0" />
-        <mass value="1.60979" />
-        <inertia ixx="0.00387607152" ixy="-0.00044384784" ixz="-0.00021115038"
-          iyy="0.00700537914" iyz="0.00015348067" izz="0.0055275524" />
-      </inertial>
-    </link>
-    <link name="right_wrist">
-      <visual>
-        <origin rpy="0 3.1416 0" xyz="0 0 0" />
-        <geometry>
-          <mesh filename="package://baxter_description/meshes/wrist/W2.STL" />
-        </geometry>
-        <material name="darkred">
-          <color rgba=".5 .1 .1 1" />
-        </material>
-      </visual>
-      <collision>
-        <origin rpy="0 3.1416 1.5708" xyz="0 0 0" />
-        <geometry>
-          <mesh filename="package://baxter_description/meshes/wrist/W2.STL" />
-        </geometry>
-      </collision>
-      <inertial>
-        <origin rpy="0 3.1416 1.5708" xyz="0.00198 0.00125 0.01855"/>
-        <mass value="0.35093" />
-        <inertia ixx="0.00025289155" ixy="0.00000575311" ixz="-0.00000159345"
-          iyy="0.0002688601" iyz="-0.00000519818" izz="0.0003074118" />
+    <!-- left_hand -->
+    <link name="left_hand">
+      <inertial>
+        <origin rpy="0 0 0" xyz="0 0 0" />
+        <mass value="0.0001" />
+        <inertia ixx="1e-08" ixy="0" ixz="0" iyy="1e-08" iyz="0" izz="1e-08" />
       </inertial>
     </link>
@@ -481,4 +497,66 @@
       <origin rpy="0 0 0" xyz="0 0 .18" />
     </joint>
+    <!-- ========== RIGHT ARM JOINTS ========== -->
+    <joint name="torso_right_upper_shoulder" type="revolute">
+      <parent link="torso" />
+      <child link="right_upper_shoulder" />
+      <origin rpy="0 0 0" xyz=".063 -.255 .025" />
+      <axis xyz="0 0 1" />
+      <limit lower="-0.89" upper="1.5708" effort="50" velocity="1.5" />
+    </joint>
+    <joint name="right_upper_shoulder_lower_shoulder" type="revolute">
+      <parent link="right_upper_shoulder" />
+      <child link="right_lower_shoulder" />
+      <origin rpy="0 0 0" xyz="0 -.075 .275" />
+      <axis xyz="1 0 0" />
+      <limit lower="-1.0472" upper="0.5236" effort="50" velocity="1.5" />
+    </joint>
+    <joint name="right_lower_shoulder_upper_elbow" type="revolute">
+      <parent link="right_lower_shoulder" />
+      <child link="right_upper_elbow" />
+      <origin rpy="0 0 0" xyz="0 -.1 0" />
+      <axis xyz="0 1 0" />
+      <limit lower="-1.5708" upper="1.5708" effort="50" velocity="1.5" />
+    </joint>
+    <joint name="right_upper_elbow_lower_elbow" type="revolute">
+      <parent link="right_upper_elbow" />
+      <child link="right_lower_elbow" />
+      <origin rpy="0 0 0" xyz="0 -.262 -.069" />
+      <axis xyz="1 0 0" />
+      <limit lower="-1.5708" upper="0.0524" effort="50" velocity="1.5" />
+    </joint>
+    <joint name="right_lower_elbow_upper_forearm" type="revolute">
+      <parent link="right_lower_elbow" />
+      <child link="right_upper_forearm" />
+      <origin rpy="0 0 0" xyz="0 0 -0.1" />
+      <axis xyz="0 0 1" />
+      <limit lower="-3.0543" upper="3.0543" effort="50" velocity="1.5" />
+    </joint>
+    <joint name="right_upper_forearm_lower_forearm" type="revolute">
+      <parent link="right_upper_forearm" />
+      <child link="right_lower_forearm" />
+      <origin rpy="0 0 0" xyz="0 .015 -.27" />
+      <axis xyz="1 0 0" />
+      <limit lower="-1.5708" upper="1.5708" effort="50" velocity="1.5" />
+    </joint>
+    <joint name="right_lower_forearm_wrist" type="revolute">
+      <parent link="right_lower_forearm" />
+      <child link="right_wrist" />
+      <origin rpy="0 0 -1.5708" xyz="0 0 -.112" />
+      <axis xyz="0 0 1" />
+      <limit lower="-3.0543" upper="3.0543" effort="50" velocity="1.5" />
+    </joint>
+    <!-- right wrist -->
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
Commit message: Remove duplicate geometry definition for electric gripper base in URDF

File: baxter_description/urdf/electric_gripper/baxter_electric_gripper.xacro (robot description, xacro)
@@ -11,8 +11,4 @@
                 <!-- <origin rpy="${-pi/2} ${pi} 0" xyz="0 0 0" /> -->
                 <origin rpy="${pi/2} 0 ${pi}" xyz="0 0 0" />
-                <geometry>
-                    <mesh
-                        filename="package://baxter_description/meshes/electric_gripper/electric_gripper_base.DAE" />
-                </geometry>
                 <geometry>
                     <mesh
