Commit message: Update README and SDF files: add troubleshooting section and adjust LiDAR joint position

File: baxter_description/urdf/sensors/lidar.urdf.xacro (robot description, xacro)
@@ -26,5 +26,5 @@
       <parent link="${parent}" />
       <child link="${frame}" />
-      <origin rpy="0 0 0" xyz="0 0 .04" />
+      <origin rpy="0 0 0" xyz="0 0 .043" />
     </joint>
   </xacro:macro>
