Commit message: URDF Refactor

File: baxter_description/urdf/baxter_standalone.urdf.xacro (robot description, xacro)
@@ -1,5 +1,5 @@
 <?xml version="1.0"?>
 <robot xmlns:xacro="http://ros.org/wiki/xacro" name="baxter">
-    <xacro:include filename="$(find baxter_description)/urdf/robots/baxter.urdf.xacro" />
+    <xacro:include filename="$(find baxter_description)/urdf/baxter.urdf.xacro" />
     <!-- Instancia para uso standalone -->
     <xacro:baxter name="baxter" use_sensors="true" />

File: baxter_description/urdf/electric_gripper/baxter_electric_gripper.xacro (robot description, xacro)
@@ -1,126 +1,126 @@
 <?xml version="1.0"?>
 <robot xmlns:xacro="http://www.ros.org/wiki/xacro" name="baxter_electric_gripper">
-    <xacro:macro name="baxter_electric_gripper"
-        params="side
-        l_finger l_finger_slot l_finger_tip l_finger_grasp
-        r_finger r_finger_slot r_finger_tip r_finger_grasp">
-        <xacro:property name="gripper_side" value="${side[0]}" scope="local" />
-        <!-- ===== BASE DEL GRIPPER ===== -->
-        <link name="${side}_gripper_base">
-            <visual>
-                <!-- <origin rpy="${-pi/2} ${pi} 0" xyz="0 0 0" /> -->
-                <origin rpy="${pi/2} 0 ${pi}" xyz="0 0 0" />
-                <geometry>
-                    <mesh
-                        filename="package://baxter_description/meshes/electric_gripper/electric_gripper_base.DAE" />
-                </geometry>
-            </visual>
-            <collision>
-                <origin rpy="${-pi/2} ${pi} 0" xyz="0.0 0.0 0" />
-                <geometry>
-                    <cylinder length="0.1" radius="0.029" />
-                </geometry>
-            </collision>
-            <inertial>
-                <origin rpy="${-pi/2} ${pi} 0" xyz="0.0 0.0 0.0" />
-                <mass value="0.3" />
-                <inertia ixx="2e-08" ixy="0" ixz="0" iyy="3e-08" iyz="0" izz="2e-08" />
-            </inertial>
-        </link>
-        <!-- ===== DEDO IZQUIERDO ===== -->
-        <xacro:property name="finger_length" value="0.0" scope="global" />
-        <xacro:include
-            filename="$(find baxter_description)/urdf/electric_gripper/fingers/${l_finger}.xacro" />
-        <xacro:finger_xacro
-            gripper_side="${gripper_side}"
-            finger_side="l"
-            reflect="1"
-            finger_tip="${l_finger_tip}"
-            finger_grasp="${l_finger_grasp}" />
-        <xacro:property name="tip_finger_length" value="${finger_length}" scope="local" />
-        <!-- ===== DEDO DERECHO ===== -->
-        <xacro:include
-            filename="$(find baxter_description)/urdf/electric_gripper/fingers/${r_finger}.xacro" />
-        <xacro:finger_xacro
-            gripper_side="${gripper_side}"
-            finger_side="r"
-            reflect="-1"
-            finger_tip="${r_finger_tip}"
-            finger_grasp="${r_finger_grasp}" />
-        <xacro:if value="${finger_length > tip_finger_length}">
-            <xacro:property name="tip_finger_length" value="${finger_length}" scope="local" />
-        </xacro:if>
-        <!-- ===== JOINT: hand → gripper_base ===== -->
-        <joint name="${side}_gripper_base_joint" type="fixed">
-            <origin rpy="0 0 0" xyz="0 0 0.025" />
-            <parent link="${side}_hand" />
-            <child link="${side}_gripper_base" />
-        </joint>
-        <!-- ===== ENDPOINT (referencia para IK / MoveIt) ===== -->
-        <link name="${side}_gripper">
-            <inertial>
-                <origin rpy="0 0 0" xyz="0 0 0" />
-                <mass value="0.0001" />
-                <inertia ixx="0" ixy="0" ixz="0" iyy="0" iyz="0" izz="0.0" />
-            </inertial>
-        </link>
-        <joint name="${side}_endpoint" type="fixed">
-            <origin rpy="0 0 0" xyz="0 0 ${tip_finger_length + 0.02}" />
-            <parent link="${side}_gripper_base" />
-            <child link="${side}_gripper" />
-        </joint>
-        <!-- ===== JOINT PRISMÁTICO: dedo izquierdo ===== -->
-        <xacro:property name="l_finger_offset"
-            value="${((l_finger_slot-1)*0.0095) - 0.011}"
-            scope="local" />
-        <joint name="${gripper_side}_gripper_l_finger_joint" type="prismatic">
-            <origin rpy="0 0 0" xyz="0.0 ${l_finger_offset} 0.02" />
-            <axis xyz="0 1 0" />
-            <parent link="${side}_gripper_base" />
-            <child link="${gripper_side}_gripper_l_finger" />
-            <limit effort="20.0" lower="0.0" upper="0.020833" velocity="5.0" />
-            <dynamics damping="0.7" friction="0.0" />
-        </joint>
-        <!-- ===== JOINT PRISMÁTICO: dedo derecho (mimic) ===== -->
-        <xacro:property name="r_finger_offset"
-            value="${((r_finger_slot-1)*-0.0095) + 0.011}"
-            scope="local" />
-        <joint name="${gripper_side}_gripper_r_finger_joint" type="prismatic">
-            <origin rpy="0 0 0" xyz="0.0 ${r_finger_offset} 0.02" />
-            <axis xyz="0 1 0" />
-            <parent link="${side}_gripper_base" />
-            <child link="${gripper_side}_gripper_r_finger" />
-            <limit effort="20.0" lower="-0.020833" upper="0.0" velocity="5.0" />
-            <mimic joint="${gripper_side}_gripper_l_finger_joint" multiplier="-1.0" />
-            <dynamics damping="0.7" friction="0.0" />
-        </joint>
-        <!-- ===== TRANSMISIONES (ROS Control) ===== -->
-        <transmission name="gripper_${side}_trans_r">
-            <type>transmission_interface/SimpleTransmission</type>
-            <joint name="${gripper_side}_gripper_r_finger_joint">
-                <hardwareInterface>hardware_interface/EffortJointInterface</hardwareInterface>
-            </joint>
-            <actuator name="gripper_${gripper_side}_motor1">
-                <hardwareInterface>hardware_interface/EffortJointInterface</hardwareInterface>
-                <mechanicalReduction>1</mechanicalReduction>
-            </actuator>
-        </transmission>
-        <transmission name="gripper_${side}_trans_l">
-            <type>transmission_interface/SimpleTransmission</type>
-            <joint name="${gripper_side}_gripper_l_finger_joint">
-                <hardwareInterface>hardware_interface/EffortJointInterface</hardwareInterface>
-            </joint>
-            <actuator name="gripper_${gripper_side}_motor2">
-                <hardwareInterface>hardware_interface/EffortJointInterface</hardwareInterface>
-                <mechanicalReduction>1</mechanicalReduction>
-            </actuator>
-        </transmission>
-        <!-- ===== GAZEBO: amortiguamiento implícito ===== -->
-        <gazebo reference="${gripper_side}_gripper_l_finger_joint">
-            <implicitSpringDamper>1</implicitSpringDamper>
-        </gazebo>
-        <gazebo reference="${gripper_side}_gripper_r_finger_joint">
-            <implicitSpringDamper>1</implicitSpringDamper>
-        </gazebo>
-    </xacro:macro>
+  <xacro:macro name="baxter_electric_gripper"
+    params="side
+    l_finger l_finger_slot l_finger_tip l_finger_grasp
+    r_finger r_finger_slot r_finger_tip r_finger_grasp">
+    <xacro:property name="gripper_side" value="${side[0]}" scope="local" />
+    <!-- ===== BASE DEL GRIPPER ===== -->
+    <link name="${side}_gripper_base">
+      <visual>
+        <!-- <origin rpy="${-pi/2} ${pi} 0" xyz="0 0 0" /> -->
+        <origin rpy="${pi/2} 0 ${pi}" xyz="0 0 0" />
+        <geometry>
+          <mesh
+            filename="package://baxter_description/meshes/electric_gripper/electric_gripper_base.DAE" />
+        </geometry>
+      </visual>
+      <collision>
+        <origin rpy="${-pi/2} ${pi} 0" xyz="0.0 0.0 0" />
+        <geometry>
+          <cylinder length="0.1" radius="0.029" />
+        </geometry>
+      </collision>
+      <inertial>
+        <origin rpy="${-pi/2} ${pi} 0" xyz="0.0 0.0 0.0" />
+        <mass value="0.3" />
+        <inertia ixx="2e-08" ixy="0" ixz="0" iyy="3e-08" iyz="0" izz="2e-08" />
+      </inertial>
+    </link>
+    <!-- ===== DEDO IZQUIERDO ===== -->
+    <xacro:property name="finger_length" value="0.0" scope="global" />
+    <xacro:include
+      filename="$(find baxter_description)/urdf/electric_gripper/fingers/${l_finger}.xacro" />
+    <xacro:finger_xacro
+      gripper_side="${gripper_side}"
+      finger_side="l"
+      reflect="1"
+      finger_tip="${l_finger_tip}"
+      finger_grasp="${l_finger_grasp}" />
+    <xacro:property name="tip_finger_length" value="${finger_length}" scope="local" />
+    <!-- ===== DEDO DERECHO ===== -->
+    <xacro:include
+      filename="$(find baxter_description)/urdf/electric_gripper/fingers/${r_finger}.xacro" />
+    <xacro:finger_xacro
+      gripper_side="${gripper_side}"
+      finger_side="r"
+      reflect="-1"
+      finger_tip="${r_finger_tip}"
+      finger_grasp="${r_finger_grasp}" />
+    <xacro:if value="${finger_length > tip_finger_length}">
+      <xacro:property name="tip_finger_length" value="${finger_length}" scope="local" />
+    </xacro:if>
+    <!-- ===== JOINT: hand → gripper_base ===== -->
+    <joint name="${side}_gripper_base_joint" type="fixed">
+      <origin rpy="0 0 0" xyz="0 0 0.025" />
+      <parent link="${side}_hand" />
+      <child link="${side}_gripper_base" />
+    </joint>
+    <!-- ===== ENDPOINT (referencia para IK / MoveIt) ===== -->
+    <link name="${side}_gripper">
+      <inertial>
+        <origin rpy="0 0 0" xyz="0 0 0" />
+        <mass value="0.0001" />
+        <inertia ixx="0" ixy="0" ixz="0" iyy="0" iyz="0" izz="0.0" />
+      </inertial>
+    </link>
+    <joint name="${side}_endpoint" type="fixed">
+      <origin rpy="0 0 0" xyz="0 0 ${tip_finger_length + 0.02}" />
+      <parent link="${side}_gripper_base" />
+      <child link="${side}_gripper" />
+    </joint>
+    <!-- ===== JOINT PRISMÁTICO: dedo izquierdo ===== -->
+    <xacro:property name="l_finger_offset"
+      value="${((l_finger_slot-1)*0.0095) - 0.011}"
+      scope="local" />
+    <joint name="${gripper_side}_gripper_l_finger_joint" type="prismatic">
+      <origin rpy="0 0 0" xyz="0.0 ${l_finger_offset} 0.02" />
+      <axis xyz="0 1 0" />
+      <parent link="${side}_gripper_base" />
+      <child link="${gripper_side}_gripper_l_finger" />
+      <limit effort="20.0" lower="0.0" upper="0.020833" velocity="5.0" />
+      <dynamics damping="0.7" friction="0.0" />
+    </joint>
+    <!-- ===== JOINT PRISMÁTICO: dedo derecho (mimic) ===== -->
+    <xacro:property name="r_finger_offset"
+      value="${((r_finger_slot-1)*-0.0095) + 0.011}"
+      scope="local" />
+    <joint name="${gripper_side}_gripper_r_finger_joint" type="prismatic">
+      <origin rpy="0 0 0" xyz="0.0 ${r_finger_offset} 0.02" />
+      <axis xyz="0 1 0" />
+      <parent link="${side}_gripper_base" />
+      <child link="${gripper_side}_gripper_r_finger" />
+      <limit effort="20.0" lower="-0.020833" upper="0.0" velocity="5.0" />
+      <mimic joint="${gripper_side}_gripper_l_finger_joint" multiplier="-1.0" />
+      <dynamics damping="0.7" friction="0.0" />
+    </joint>
+    <!-- ===== TRANSMISIONES (ROS Control) ===== -->
+    <transmission name="gripper_${side}_trans_r">
+      <type>transmission_interface/SimpleTransmission</type>
+      <joint name="${gripper_side}_gripper_r_finger_joint">
+        <hardwareInterface>hardware_interface/EffortJointInterface</hardwareInterface>
+      </joint>
+      <actuator name="gripper_${gripper_side}_motor1">
+        <hardwareInterface>hardware_interface/EffortJointInterface</hardwareInterface>
+        <mechanicalReduction>1</mechanicalReduction>
+      </actuator>
+    </transmission>
+    <transmission name="gripper_${side}_trans_l">
+      <type>transmission_interface/SimpleTransmission</type>
+      <joint name="${gripper_side}_gripper_l_finger_joint">
+        <hardwareInterface>hardware_interface/EffortJointInterface</hardwareInterface>
+      </joint>
+      <actuator name="gripper_${gripper_side}_motor2">
+        <hardwareInterface>hardware_interface/EffortJointInterface</hardwareInterface>
+        <mechanicalReduction>1</mechanicalReduction>
+      </actuator>
+    </transmission>
+    <!-- ===== GAZEBO AMORTIGUAMIENTO IMPLICITO ===== -->
+    <gazebo reference="${gripper_side}_gripper_l_finger_joint">
+      <implicitSpringDamper>1</implicitSpringDamper>
+    </gazebo>
+    <gazebo reference="${gripper_side}_gripper_r_finger_joint">
+      <implicitSpringDamper>1</implicitSpringDamper>
+    </gazebo>
+  </xacro:macro>
 </robot>

File: gazebo_baxter/urdf/baxter_gazebo.urdf.xacro (robot description, xacro)
@@ -2,5 +2,5 @@
 <robot xmlns:xacro="http://ros.org/wiki/xacro" name="baxter">
   <!-- Include pure robot -->
-  <xacro:include filename="$(find baxter_description)/urdf/robots/baxter.urdf.xacro" />
+  <xacro:include filename="$(find baxter_description)/urdf/baxter.urdf.xacro" />
   <!-- Include gazebo sensors -->
   <xacro:include filename="$(find gazebo_baxter)/urdf/sensors/imu_gazebo.urdf.xacro" />
